Commit message: Swap drone models to gym-pybullet-drones research URDFs
- interceptor.urdf: cf2x Crazyflie quadrotor (research-grade geometry)
- intruder.urdf: racer quadrotor scaled 3x (loitering munition stand-in)
- cf2.dae: shared Crazyflie mesh referenced by both URDFs
- Drone default URDF updated to interceptor.urdf
- LoiteringMunition loads with globalScaling=3.0 for threat visibility
- Red tint (all links) applied to LoiteringMunition after load
- Blue tint handled by existing Drone._apply_color("blue") path

Co-Authored-By: Claude Sonnet 4.6 <noreply@anthropic.com>

File: anti-drone-dome/assets/interceptor.urdf (robot description, URDF)
Before this commit: robot interceptor_quad, 13 links, 12 joints
Links:
- removed link arm_0
- removed link arm_1
- removed link arm_2
- removed link arm_3
- removed link gear_bl
- removed link gear_br
- removed link gear_fl
- removed link gear_fr
- removed link rotor_0
- removed link rotor_1
- removed link rotor_2
- removed link rotor_3
- added link center_of_mass_link, mass 0
- added link prop0_link, mass 0
- added link prop1_link, mass 0
- added link prop2_link, mass 0
- added link prop3_link, mass 0
- link base_link: mass 1.5 -> 0.027; geometry collision cylinder length=.025 radius=.06; visual mesh filename=./cf2.dae scale=1 1 1
Joints:
- removed joint arm_0_joint
- removed joint arm_1_joint
- removed joint arm_2_joint
- removed joint arm_3_joint
- removed joint gear_bl_joint
- removed joint gear_br_joint
- removed joint gear_fl_joint
- removed joint gear_fr_joint
- removed joint rotor_0_joint
- removed joint rotor_1_joint
- removed joint rotor_2_joint
- removed joint rotor_3_joint
- added joint center_of_mass_joint: type fixed, parent base_link, child center_of_mass_link
- added joint prop0_joint: type fixed, parent base_link, child prop0_link
- added joint prop1_joint: type fixed, parent base_link, child prop1_link
- added joint prop2_joint: type fixed, parent base_link, child prop2_link
- added joint prop3_joint: type fixed, parent base_link, child prop3_link

File: anti-drone-dome/assets/intruder.urdf (robot description, URDF)
Before this commit: robot loitering_munition, 9 links, 8 joints
Links:
- removed link nose
- removed link rotor_arm
- removed link rotor_left
- removed link rotor_right
- removed link tail_horiz
- removed link tail_vert
- removed link wing_left
- removed link wing_right
- added link center_of_mass_link, mass 0
- added link prop0_link, mass 0
- added link prop1_link, mass 0
- added link prop2_link, mass 0
- added link prop3_link, mass 0
- link base_link: mass 1.2 -> 0.830; geometry collision cylinder length=.025 radius=.06; visual mesh filename=./cf2.dae scale=3 3 3
Joints:
- removed joint nose_joint
- removed joint rotor_arm_joint
- removed joint rotor_left_joint
- removed joint rotor_right_joint
- removed joint tail_horiz_joint
- removed joint tail_vert_joint
- removed joint wing_left_joint
- removed joint wing_right_joint
- added joint center_of_mass_joint: type fixed, parent base_link, child center_of_mass_link
- added joint prop0_joint: type fixed, parent base_link, child prop0_link
- added joint prop1_joint: type fixed, parent base_link, child prop1_link
- added joint prop2_joint: type fixed, parent base_link, child prop2_link
- added joint prop3_joint: type fixed, parent base_link, child prop3_link

Commit message: Build integrated tactical simulation and validation workbench
Add realistic scenarios, fused radar/EO sensing, residual-RL training and evidence-backed tactical views. Introduce safe hardware profiles, mission recording, SIL/HIL validation reports, OpenGL rendering selection, and explicit CUDA device controls.

Co-authored-by: Copilot <223556219+Copilot@users.noreply.github.com>

File: anti-drone-dome/assets/interceptor.urdf (robot description, URDF)
Before this commit: robot cf2, 6 links, 5 joints
Links:
- removed link center_of_mass_link
- removed link prop0_link
- removed link prop1_link
- removed link prop2_link
- removed link prop3_link
- added link left_fin, mass 0; visual box size=0.58 0.72 0.06
- added link lower_fin, mass 0; visual box size=0.44 0.06 0.48
- added link nose, mass 0; visual sphere radius=0.13
- added link right_fin, mass 0; visual box size=0.58 0.72 0.06
- added link upper_fin, mass 0; visual box size=0.44 0.06 0.48
- link base_link: mass 0.027 -> 0.83; geometry collision box size=1.55 0.35 0.30; visual cylinder length=1.55 radius=0.13
Joints:
- removed joint center_of_mass_joint
- removed joint prop0_joint
- removed joint prop1_joint
- removed joint prop2_joint
- removed joint prop3_joint
- added joint left_fin_joint: type fixed, parent base_link, child left_fin
- added joint lower_fin_joint: type fixed, parent base_link, child lower_fin
- added joint nose_joint: type fixed, parent base_link, child nose
- added joint right_fin_joint: type fixed, parent base_link, child right_fin
- added joint upper_fin_joint: type fixed, parent base_link, child upper_fin
